File: KICAD/CM400T_CDI_Revision_A/CM400T_CDI_Revision_A.kicad_pcb (KiCad board)
At the start: 2 copper layers, 66.4 x 46 mm, 42 parts, among them P1 Brown, P2 Green Coil, P3 Black w/ White, P4 Yellow Coil, P5 Blue, P6 White, P7 Light Blue, P8 Green Harness, P9 Pink

Commit message: make rev a schematic more readable.
Parts:
- R2: value R_US -> 1M
- R3: value R_US -> 22
- R4: value 2.7K -> 3.3K
- R5: value 1.8K -> 56
Changed lines of the file:
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@@
       (effects (font (size 1 1) (thickness 0.15)))
     )
-    (fp_text value "1.8K" (at 5.08 2.37) (layer "F.Fab")
+    (fp_text value "56" (at 5.08 2.37) (layer "F.Fab")
       (effects (font (size 1 1) (thickness 0.15)))
     )
@@
     (fp_line (start 4.23 1.42) (end 31.115 1.42) (layer "F.SilkS") (width 0.12))
     (fp_line (start 15.875 0) (end 4.23 0) (layer "F.SilkS") (width 0.12))
-    (fp_line (start 33.655 0) (end 18.415 0) (layer "F.SilkS") (width 0.12))
     (fp_line (start 4.23 -1.42) (end 4.23 1.42) (layer "F.SilkS") (width 0.12))
     (fp_line (start 31.115 -1.42) (end 4.23 -1.42) (layer "F.SilkS") (width 0.12))
+    (fp_line (start 33.655 0) (end 18.415 0) (layer "F.SilkS") (width 0.12))
     (fp_line (start 1.04 0) (end 4.23 0) (layer "F.SilkS") (width 0.12))
     (fp_line (start -1.05 -1.55) (end -1.05 1.55) (layer "F.CrtYd") (width 0.05))
@@
     (fp_line (start 36.195 -1.55) (end -1.05 -1.55) (layer "F.CrtYd") (width 0.05))
     (fp_line (start -1.05 1.55) (end 36.195 1.55) (layer "F.CrtYd") (width 0.05))
+    (fp_line (start 18.415 0) (end 18.415 0) (layer "F.Fab") (width 0.1))
     (fp_line (start 4.35 -1.3) (end 4.35 1.3) (layer "F.Fab") (width 0.1))
     (fp_line (start 0 0) (end 4.35 0) (layer "F.Fab") (width 0.1))
@@
     (fp_line (start 4.35 1.3) (end 31.115 1.3) (layer "F.Fab") (width 0.1))
     (fp_line (start 15.875 0) (end 4.35 0) (layer "F.Fab") (width 0.1))
+    (fp_line (start 15.875 0) (end 15.875 0) (layer "F.Fab") (width 0.1))
+    (fp_line (start 31.115 -1.3) (end 4.35 -1.3) (layer "F.Fab") (width 0.1))
     (fp_line (start 34.29 0) (end 18.415 0) (layer "F.Fab") (width 0.1))
-    (fp_line (start 15.875 0) (end 15.875 0) (layer "F.Fab") (width 0.1))
-    (fp_line (start 18.415 0) (end 18.415 0) (layer "F.Fab") (width 0.1))
-    (fp_line (start 31.115 -1.3) (end 4.35 -1.3) (layer "F.Fab") (width 0.1))
     (pad "1" thru_hole circle (at 0 0) (size 1.6 1.6) (drill 0.8) (layers *.Cu *.Mask)
       (net 2 "Net-(C1-Pad1)") (pintype "passive"))
@@
       (effects (font (size 1 1) (thickness 0.15)))
     )
-    (fp_text value "R_US" (at 5.08 2.37) (layer "F.Fab")
+    (fp_text value "22" (at 5.08 2.37) (layer "F.Fab")
       (effects (font (size 1 1) (thickness 0.15)))
     )
@@
       (effects (font (size 1 1) (thickness 0.15)))
     )
-    (fp_text value "2.7K" (at 5.08 2.37) (layer "F.Fab")
+    (fp_text value "3.3K" (at 5.08 2.37) (layer "F.Fab")
       (effects (font (size 1 1) (thickness 0.15)))
     )
@@
       (effects (font (size 1 1) (thickness 0.15)))
     )
-    (fp_text value "R_US" (at 5.08 2.37) (layer "F.Fab")
+    (fp_text value "1M" (at 5.08 2.37) (layer "F.Fab")
       (effects (font (size 1 1) (thickness 0.15)))
     )
@@
   (segment (start 155.83 118.5) (end 159.08 115.25) (width 1.524) (layer "B.Cu") (net 3))
   (segment (start 159.08 115.25) (end 159.08 111) (width 1.524) (layer "B.Cu") (net 3))
-  (segment (start 159.08 111) (end 159.33 110.75) (width 1.524) (layer "B.Cu") (net 3))
   (segment (start 170.195 113.96) (end 167.96 113.96) (width 1.524) (layer "B.Cu") (net 3))
   (segment (start 153.33 118.5) (end 155.83 118.5) (width 1.524) (layer "B.Cu") (net 3))
@@
   (segment (start 159.33 110.75) (end 162.75 110.75) (width 1.524) (layer "B.Cu") (net 3))
   (segment (start 122.75 86.75) (end 122.75 98.42) (width 1.524) (layer "B.Cu") (net 4))
-  (segment (start 122.75 98.42) (end 122.67 98.5) (width 1.524) (layer "B.Cu") (net 4))
   (segment (start 164.83 103.67) (end 163.75 104.75) (width 1.524) (layer "B.Cu") (net 5))
   (segment (start 164.83 101.5) (end 164.83 103.67) (width 1.524) (layer "B.Cu") (net 5))
@@
   (segment (start 172.43304 107.25) (end 172.59152 107.40848) (width 1.524) (layer "B.Cu") (net 6))
   (segment (start 170.195 116.5) (end 171.024515 116.5) (width 1.524) (layer "B.Cu") (net 6))
-  (segment (start 165.175 94.405) (end 165.08 94.5) (width 1.524) (layer "B.Cu") (net 6))
   (segment (start 172.59152 114.932995) (end 172.59152 107.40848) (width 1.524) (layer "B.Cu") (net 6))
   (segment (start 169.5 107.25) (end 172.43304 107.25) (width 1.524) (layer "B.Cu") (net 6))
@@
   (segment (start 171.024515 116.5) (end 172.59152 114.932995) (width 1.524) (layer "B.Cu") (net 6))
   (segment (start 172.59152 107.40848) (end 172.59152 97.09152) (width 1.524) (layer "B.Cu") (net 6))
-  (segment (start 165.1025 94.4775) (end 165.08 94.5) (width 1.524) (layer "B.Cu") (net 6))
   (segment (start 165.08 97.92) (end 165.16 98) (width 1.524) (layer "B.Cu") (net 6))
   (segment (start 165.33 80) (end 165.33 84.25) (width 1.524) (layer "B.Cu") (net 6))

Commit message: Clean up Rev A PCB a bit.
Parts:
- moved H2 60.4 mm to (168.8, 100.0)
- moved H1 36.0 mm to (145.5, 102.8)
- moved H4 35.6 mm to (113.8, 104.5)
- moved H3 25.2 mm to (168.8, 89.5)
- moved R4 2.37 mm to (143.9, 116.2)
- moved R10 2.26 mm to (149.2, 113.0)
- moved C5 2.25 mm to (146.5, 113.0)
- moved R5 2.25 mm to (140.8, 116.2)
- moved R7 1.78 mm to (130.6, 113.0)
- moved R8 1.52 mm to (130.6, 109.2)
- moved C3 1.50 mm to (139.2, 109.2)
- moved D5 1.50 mm to (159.3, 109.2)
- moved P7 1.50 mm to (144.8, 109.2)
- moved R2 1.41 mm to (164.6, 119.8)
- moved SCR1 1.25 mm to (170.2, 117.8)
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Routing:
- net Net-(C1-Pad2): track 67.3 -> 77.1 mm
- net Net-(C5-Pad1): track 34.9 -> 31.2 mm
- net Net-(C3-Pad2): track 182.6 -> 179.0 mm
- net Net-(C4-Pad2): track 50.8 -> 48.3 mm
- net Net-(D5-Pad1): track 24.4 -> 22.6 mm
- net Net-(R7-Pad2): track 8.58 -> 9.35 mm
- net Net-(R5-Pad1): track 2.34 -> 3.09 mm
Other:
- board size 66.4 x 46 mm -> 67.1 x 46 mm
